Commit message: second version

File: ai_robot_ranger_mini/ranger_mini_gazebo/xacro/ranger_mini_sensors.xacro (robot description, xacro)
@@ -196,63 +196,5 @@
     </plugin>
   </gazebo>
-  <!--kinect camera-->
-  <link name="kinect_link">
-    <visual>
-      <origin rpy="0 0 0" xyz="0 0 0"/>
-      <geometry>
-        <mesh filename="package://ranger_mini_gazebo/description/meshes/xtion/asus_xtion_pro_camera.dae"/>
-      </geometry>
-    </visual>
-    <inertial>
-        <mass value="0.0001" />
-        <origin xyz="0 0 0" />
-        <inertia ixx="0.0001" ixy="0.0" ixz="0.0"
-                 iyy="0.0001" iyz="0.0"
-                 izz="0.0001" />
-    </inertial>
-  </link>
-  <joint name="base_kinect_joint" type="fixed">
-    <origin rpy="0 0 0" xyz="0.24376 -0.012728 0.475118"/>
-    <parent link="base_link"/>
-    <child link="kinect_link"/>
-  </joint>
-  <gazebo reference="kinect_link">
-   <sensor type="depth" name="kinect">
-    <alwaysOn>true</alwaysOn>
-    <updateRate>10</updateRate>
-    <camera>
-          <horizontal_fov>1.57</horizontal_fov>
-          <image>
-            <format>R8G8B8</format>
-            <width>640</width>
-            <height>480</height>
-          </image>
-          <clip>
-            <near>0.05</near>
-            <far>10.0</far>
-          </clip>
-    </camera>
-    <plugin name="kinect_controller" filename="libgazebo_ros_openni_kinect.so">
-      <baseline>0.2</baseline>
-      <cameraName>kinect_ir</cameraName>
-      <imageTopicName>/kinect/rgb/image_raw</imageTopicName>
-      <cameraInfoTopicName>/kinect/rgb/camera_info</cameraInfoTopicName>
-      <depthImageTopicName>/kinect/depth/image_raw</depthImageTopicName>
-      <depthImageInfoTopicName>/kinect/depth/camera_info</depthImageInfoTopicName>
-      <pointCloudTopicName>/kinect/depth/points</pointCloudTopicName>
-      <frameName>kinect_link</frameName>
-      <pointCloudCutoff>0.5</pointCloudCutoff>
-      <distortionK1>0.00000001</distortionK1>
-      <distortionK2>0.00000001</distortionK2>
-      <distortionK3>0.00000001</distortionK3>
-      <distortionT1>0.00000001</distortionT1>
-      <distortionT2>0.00000001</distortionT2>
-      <CxPrime>0</CxPrime>
-      <Cx>0</Cx>
-      <Cy>0</Cy>
-      <focalLength>0</focalLength>
-      <hackBaseline>0</hackBaseline>
-    </plugin>
-   </sensor>
-  </gazebo>
+  <!-- ZED2 sim -->
+  <xacro:include filename="$(find ranger_mini_gazebo)/xacro/zed2.xacro"/>
 </robot>

Commit message: third version

File: ai_robot_ranger_mini/ranger_mini_gazebo/xacro/ranger_mini_sensors.xacro (robot description, xacro)
@@ -2,4 +2,54 @@
 <robot name="ranger_mini" xmlns:controller="http://playerstage.sourceforge.net/gazebo/xmlschema/#controller" xmlns:interface="http://playerstage.sourceforge.net/gazebo/xmlschema/#interface" xmlns:sensor="http://playerstage.sourceforge.net/gazebo/xmlschema/#sensor" xmlns:xacro="http://ros.org/wiki/xacro">
   <!-- Lidar sim -->
+ <!--link name="velodyne">
+    <inertial>
+      <mass value="0.01"/>
+      <origin xyz="0 0 0"/>
+      <inertia ixx="1e-7" ixy="0.0" ixz="0.0" iyy="1e-7" iyz="0.0" izz="1e-7"/>
+    </inertial>
+    <visual>
+      <origin xyz="0 0 0" rpy="0 0 0"/>
+        <geometry>
+          <mesh filename="package://ranger_mini_gazebo/description/meshes/velodyne_hdl32/velodyne_base.dae" />
+        </geometry>
+      </visual>
+  </link>
+  <gazebo reference="velodyne">
+    <sensor name="sensor_velodyne" type="ray">
+	<visualize>0</visualize>
+	<update_rate>10</update_rate>
+	<pose> 0 0 0 0 0 0 </pose>
+	<plugin name="ros_velodyne" filename="libgazebo_ros_velodyne_laser.so">
+          <topicName>/points</topicName>
+          <frameName>velodyne</frameName>
+	</plugin>
+	<ray>
+	  <scan>
+            <horizontal>
+            	<samples>100</samples>
+            	<resolution>1</resolution>
+            	<min_angle>-2.356194</min_angle>
+            	<max_angle>2.356194</max_angle>
+            </horizontal>
+            <vertical>
+            	<samples>16</samples>
+            	<resolution>1</resolution>
+            	<min_angle>-0.261799</min_angle>
+            	<max_angle>0.261799</max_angle>
+            </vertical>
+          </scan>
+	  <range>
+          	<min>0.10</min>
+          	<max>20.0</max>
+          	<resolution>0.001</resolution>
+          </range>
+	</ray>
+    </sensor>
+  </gazebo>
+  <joint name="base_velodyne_joint" type="fixed">
+    <origin rpy="0 0 0" xyz="0.21386 -0.0094087 0.581"/>
+    <parent link="base_link"/>
+    <child link="velodyne"/>
+  </joint-->
   <joint name="hokuyo_joint" type="fixed">
     <axis xyz="0 0 0" />
@@ -196,5 +246,69 @@
     </plugin>
   </gazebo>
-  <!-- ZED2 sim -->
-  <xacro:include filename="$(find ranger_mini_gazebo)/xacro/zed2.xacro"/>
+  <!--kinect camera-->
+  <link name="kinect_link">
+    <visual>
+      <origin rpy="0 0 0" xyz="0 0 0"/>
+      <geometry>
+        <mesh filename="package://ranger_mini_gazebo/description/meshes/xtion/asus_xtion_pro_camera.dae"/>
+      </geometry>
+    </visual>
+    <inertial>
+        <mass value="0.0001" />
+        <origin xyz="0 0 0" />
+        <inertia ixx="0.0001" ixy="0.0" ixz="0.0"
+                 iyy="0.0001" iyz="0.0"
+                 izz="0.0001" />
+    </inertial>
+  </link>
+  <joint name="base_kinect_joint" type="fixed">
+    <origin rpy="0 0 0" xyz="0.24376 -0.012728 0.475118"/>
+    <parent link="base_link"/>
+    <child link="kinect_link"/>
+  </joint>
+  <link name="camera_link_fake"/>
+  <joint name="camera_joint_fake" type="fixed">
+    <origin xyz="0 0 0" rpy="-1.5708 0 -1.5708"/>
+    <parent link="kinect_link"/>
+    <child link="camera_link_fake"/>
+  </joint>
+  <gazebo reference="kinect_link">
+   <sensor type="depth" name="kinect">
+    <alwaysOn>true</alwaysOn>
+    <updateRate>10</updateRate>
+    <camera>
+          <horizontal_fov>1.57</horizontal_fov>
+          <image>
+            <format>R8G8B8</format>
+            <width>640</width>
+            <height>480</height>
+          </image>
+          <clip>
+            <near>0.05</near>
+            <far>10.0</far>
+          </clip>
+    </camera>
+    <plugin name="kinect_controller" filename="libgazebo_ros_openni_kinect.so">
+      <baseline>0.2</baseline>
+      <cameraName>kinect_ir</cameraName>
+      <imageTopicName>/kinect/rgb/image_raw</imageTopicName>
+      <cameraInfoTopicName>/kinect/rgb/camera_info</cameraInfoTopicName>
+      <depthImageTopicName>/kinect/depth/image_raw</depthImageTopicName>
+      <depthImageInfoTopicName>/kinect/depth/camera_info</depthImageInfoTopicName>
+      <pointCloudTopicName>/kinect/depth/points</pointCloudTopicName>
+      <frameName>camera_link_fake</frameName>
+      <pointCloudCutoff>0.5</pointCloudCutoff>
+      <distortionK1>0.00000001</distortionK1>
+      <distortionK2>0.00000001</distortionK2>
+      <distortionK3>0.00000001</distortionK3>
+      <distortionT1>0.00000001</distortionT1>
+      <distortionT2>0.00000001</distortionT2>
+      <CxPrime>0</CxPrime>
+      <Cx>0</Cx>
+      <Cy>0</Cy>
+      <focalLength>0</focalLength>
+      <hackBaseline>0</hackBaseline>
+    </plugin>
+   </sensor>
+  </gazebo>
 </robot>
