Commit message: fourth version

File: ai_robot_ranger_mini/ranger_mini_gazebo/xacro/pioneer3at.urdf (robot description, URDF)
Before this commit: robot pioneer3at, 11 links, 10 joints
Links:
- link base_link: mass 1.798 -> 3.798
Joints:
- joint base_link2base_footprint: origin xyz=0 0 0.2 -> xyz=0 0 -0.2

File: ai_robot_ranger_mini/ranger_mini_gazebo/xacro/ranger_mini.gazebo.xacro (robot description, xacro)
@@ -3,4 +3,5 @@
 <!-- Gazebo references -->
 <gazebo reference="base_link">
+  <gravity>true</gravity>
   <mu1 value="0.1"/>
   <mu2 value="0.1"/>
@@ -9,51 +10,59 @@
   <material>Gazebo/White</material>
 </gazebo>
-	<gazebo reference="front_left_steering_link">
-	  <!-- <selfCollide>false</selfCollide> -->
-      <mu1 value="1.5" />
-      <mu2 value="1.5" />
-     <material>Gazebo/Grey</material>
-    </gazebo>
-	<gazebo reference="front_right_steering_link">
-	  <!-- <selfCollide>false</selfCollide> -->
-      <mu1 value="1.5" />
-      <mu2 value="1.5" />
-      <material>Gazebo/Grey</material>
-    </gazebo>
-  	<gazebo reference="rear_left_steering_link">
-	  <!-- <selfCollide>false</selfCollide> -->
-      <mu1 value="1.5" />
-      <mu2 value="1.5" />
-      <material>Gazebo/Grey</material>
-    </gazebo>
-  	<gazebo reference="rear_right_steering_link">
-	  <!-- <selfCollide>false</selfCollide> -->
-      <mu1 value="1.5" />
-      <mu2 value="1.5" />
-      <material>Gazebo/Grey</material>
-    </gazebo>
-    <gazebo reference="ffl_wheel_link">
-      <!-- <selfCollide>false</selfCollide> -->
-      <mu1 value="0.1" />
-      <mu2 value="0.1" />
-      <material>Gazebo/Grey</material>
-    </gazebo>
-    <gazebo reference="ffr_wheel_link">
-      <!-- <selfCollide>false</selfCollide> -->
-      <mu1 value="0.1" />
-      <mu2 value="0.1" />
-      <material>Gazebo/Grey</material>
-    </gazebo>
-    <gazebo reference="rfl_wheel_link">
-      <!-- <selfCollide>false</selfCollide> -->
-      <mu1 value="0.1" />
-      <mu2 value="1.1" />
-      <material>Gazebo/Grey</material>
-    </gazebo>
-    <gazebo reference="rfr_wheel_link">
-      <!-- <selfCollide>false</selfCollide> -->
-      <mu1 value="0.1" />
-      <mu2 value="0.1" />
-      <material>Gazebo/Grey</material>
-    </gazebo>
+<gazebo reference="front_left_steering_link">
+  <!-- <selfCollide>false</selfCollide> -->
+  <gravity>true</gravity>
+  <mu1 value="1.5" />
+  <mu2 value="1.5" />
+  <material>Gazebo/Grey</material>
+</gazebo>
+<gazebo reference="front_right_steering_link">
+  <!-- <selfCollide>false</selfCollide> -->
+  <gravity>true</gravity>
+  <mu1 value="1.5" />
+  <mu2 value="1.5" />
+  <material>Gazebo/Grey</material>
+</gazebo>
+<gazebo reference="rear_left_steering_link">
+  <!-- <selfCollide>false</selfCollide> -->
+  <gravity>true</gravity>
+  <mu1 value="1.5" />
+  <mu2 value="1.5" />
+  <material>Gazebo/Grey</material>
+</gazebo>
+<gazebo reference="rear_right_steering_link">
+  <!-- <selfCollide>false</selfCollide> -->
+  <gravity>true</gravity>
+  <mu1 value="1.5" />
+  <mu2 value="1.5" />
+  <material>Gazebo/Grey</material>
+</gazebo>
+<gazebo reference="ffl_wheel_link">
+  <!-- <selfCollide>false</selfCollide> -->
+  <gravity>true</gravity>
+  <mu1 value="0.1" />
+  <mu2 value="0.1" />
+  <material>Gazebo/Grey</material>
+</gazebo>
+<gazebo reference="ffr_wheel_link">
+  <!-- <selfCollide>false</selfCollide> -->
+  <gravity>true</gravity>
+  <mu1 value="0.1" />
+  <mu2 value="0.1" />
+  <material>Gazebo/Grey</material>
+</gazebo>
+<gazebo reference="rfl_wheel_link">
+  <!-- <selfCollide>false</selfCollide> -->
+  <gravity>true</gravity>
+  <mu1 value="0.1" />
+  <mu2 value="1.1" />
+  <material>Gazebo/Grey</material>
+</gazebo>
+<gazebo reference="rfr_wheel_link">
+  <!-- <selfCollide>false</selfCollide> -->
+  <gravity>true</gravity>
+  <mu1 value="0.1" />
+  <mu2 value="0.1" />
+  <material>Gazebo/Grey</material>
+</gazebo>
 </robot>
